File: arduino-mega-2560.kicad_sch (KiCad schematic)
At the start: 71 parts, among them J1 USB_B, J10 Conn_02x18_Odd_Even, J11 Conn_01x08, J12 Conn_PIC_ICSP_ICD, J2 Conn_02x02_Odd_Even, J3 Conn_02x03_Top_Bottom, J4 Conn_01x08, J5 Conn_01x08, J6 Conn_01x08, J7 Conn_01x10, J8 Conn_PIC_ICSP_ICD, J9 Conn_01x08, SW2 SW_MEC_5E, U1 MCU-ATMEGA2560-16AU_TQFP100_, U3 ATmega16U2-A, U5 LMV358, U6 LP2985-3.3, U8 LD1117S50CTR, Y2 CSTCE16M9V53-R0, Y3 Crystal

Commit message: halfway through labelling
Parts:
- removed C10, C11, C15, C16, C17, C18, C19, C20, C3, C4, C5, C6, C7, C8, C9: C_Small, symbol Device:C_Small
- removed C12, C13, C14: C_Polarized, symbol Device:C_Polarized
- removed D1, D5, D7: D, symbol Device:D
- removed D2, D3, D4, D6: LED, symbol Device:LED
- removed F1: MF-MSMF050-2, FUSE_F050-2, symbol MF_MSMF050_2:MF-MSMF050-2
- removed J1: USB_B, symbol Connector:USB_B
- removed J10: Conn_02x18_Odd_Even, symbol Connector_Generic:Conn_02x18_Odd_Even
- removed J11, J4, J5, J6, J9: Conn_01x08, symbol Connector_Generic:Conn_01x08
- removed J12, J8: Conn_PIC_ICSP_ICD, symbol Connector:Conn_PIC_ICSP_ICD
- removed J2: Conn_02x02_Odd_Even, symbol Connector_Generic:Conn_02x02_Odd_Even
- removed J3: Conn_02x03_Top_Bottom, symbol Connector_Generic:Conn_02x03_Top_Bottom
- removed J7: Conn_01x10, symbol Connector_Generic:Conn_01x10
- removed L1: MH2029-300Y, IND_BOURNS_MH2029, symbol MH2029_300Y:MH2029-300Y
- removed R1, R10, R11, R12, R13, R14, R15, R16, R17, R18, R19, R2, R20, R21, R22, R3, R4, R5, R6, R7, R8, R9: R, symbol Device:R
- removed RV1, RV2: Varistor, symbol Device:Varistor
- removed SW2: SW_MEC_5E, symbol Switch:SW_MEC_5E
- removed U1: MCU-ATMEGA2560-16AU_TQFP100_, MCU-ATMEGA2560-16AU_TQFP100_:TQFP100-0.5-14X14MM, symbol MCU-ATMEGA2560-16AU_TQFP100_:MCU-ATMEGA2560-16AU_TQFP100_
- removed U3: ATmega16U2-A, Package_QFP:TQFP-32_7x7mm_P0.8mm, symbol MCU_Microchip_ATmega:ATmega16U2-A
- removed U5: LMV358, symbol Amplifier_Operational:LMV358
- removed U6: LP2985-3.3, Package_TO_SOT_SMD:SOT-23-5, symbol Regulator_Linear:LP2985-3.3
- removed U8: LD1117S50CTR, LD1117S50CTR:SOT230P700X180-4N, symbol LD1117S50CTR:LD1117S50CTR
- removed Y2: CSTCE16M9V53-R0, CSTCE16M9V53-R0:OSC_CSTCE16M9V53-R0, symbol CSTCE16M9V53-R0:CSTCE16M9V53-R0
- removed Y3: Crystal, symbol Device:Crystal
Other:
- added sheet ATmega16U2 (ATmega16U2.kicad_sch)
- added sheet MCU-ATMEGA2560 (MCU-ATMEGA2560.kicad_sch)
- added sheet power-supply (power-supply.kicad_sch)

Commit message: hardest trial
Other:
- added sheet Mounting Holes (mountingHoles.kicad_sch)
Changed lines of the file:
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@@
+	)
+	(sheet
+		(at 31.75 106.68)
+		(size 71.12 62.23)
+		(fields_autoplaced yes)
+		(stroke
+			(width 0.1524)
+			(type solid)
+		)
+		(fill
+			(color 0 0 0 0.0000)
+		)
+		(property "Sheetname" "Mounting Holes"
+			(at 31.75 105.9684 0)
+			(effects
+				(font
+					(size 1.27 1.27)
+				)
+				(justify left bottom)
+			)
+		)
+		(property "Sheetfile" "mountingHoles.kicad_sch"
+			(at 31.75 169.4946 0)
+			(effects
+				(font
+					(size 1.27 1.27)
+				)
+				(justify left top)
+			)
+		)
+		(instances
+			(project "arduino-mega-2560"
+				(path "/01593c05-32ee-43cc-9d3f-a6fed62a39f4"
+					(page "5")
+				)
+			)
+		)
 	)
 	(sheet
