File: MCU-ATMEGA2560.kicad_sch (KiCad schematic)
At the start: 40 parts, among them J10 Conn_01x10, J15 Conn_02x03_Odd_Even, J4 Conn_02x18_Odd_Even, J5 Conn_01x08, J6 Conn_01x08, J7 Conn_01x08, J8 Conn_01x08, J9 Conn_01x08, SW1 SW_MEC_5E, U1 LMV358, U4 MCU-ATMEGA2560-16AU_TQFP100_, U5 LP2985-3.3, U6 PMV48XP, Y1 CSTCE16M9V53-R0

Commit message: finished ratsnests connections
Changed lines of the file:
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@@
 	)
 	(junction
-		(at 59.69 250.19)
-		(diameter 0)
-		(color 0 0 0 0)
-	)
-	(junction
 		(at 132.08 101.6)
 		(diameter 0)
@@
 	)
 	(junction
+		(at 59.69 250.19)
+		(diameter 0)
+		(color 0 0 0 0)
+	)
+	(junction
 		(at 92.71 93.98)
 		(diameter 0)
@@
 	(wire
 		(pts
-			(xy 59.69 250.19) (xy 59.69 254)
-		)
-		(stroke
-			(width 0)
-			(type default)
-		)
-	)
-	(wire
-		(pts
 			(xy 52.07 228.6) (xy 52.07 233.68)
 		)
@@
 	(wire
 		(pts
-			(xy 30.48 247.65) (xy 36.83 247.65)
-		)
-		(stroke
-			(width 0)
-			(type default)
-		)
-	)
-	(wire
-		(pts
 			(xy 259.08 24.13) (xy 259.08 36.83)
 		)
@@
 	(wire
 		(pts
-			(xy 52.07 250.19) (xy 59.69 250.19)
+			(xy 59.69 250.19) (xy 52.07 250.19)
 		)
 		(stroke
@@
 	(wire
 		(pts
-			(xy 59.69 250.19) (xy 66.04 250.19)
-		)
-		(stroke
-			(width 0)
-			(type default)
-		)
-	)
-	(wire
-		(pts
 			(xy 109.22 242.57) (xy 120.65 242.57)
 		)
@@
 	(wire
 		(pts
+			(xy 66.04 250.19) (xy 59.69 250.19)
+		)
+		(stroke
+			(width 0)
+			(type default)
+		)
+	)
+	(wire
+		(pts
 			(xy 100.33 129.54) (xy 100.33 124.46)
 		)
@@
 	(wire
 		(pts
-			(xy 203.2 234.95) (xy 203.2 240.03)
-		)
-		(stroke
-			(width 0)
-			(type default)
-		)
-	)
-	(wire
-		(pts
 			(xy 226.06 109.22) (xy 233.68 109.22)
 		)
@@
 	(wire
 		(pts
+			(xy 30.48 247.65) (xy 36.83 247.65)
+		)
+		(stroke
+			(width 0)
+			(type default)
+		)
+	)
+	(wire
+		(pts
 			(xy 54.61 129.54) (xy 60.96 129.54)
 		)
@@
 	(wire
 		(pts
-			(xy 30.48 247.65) (xy 30.48 251.46)
-		)
-		(stroke
-			(width 0)
-			(type default)
-		)
-	)
-	(wire
-		(pts
 			(xy 232.41 157.48) (xy 232.41 153.67)
 		)
@@
 		)
 	)
-	(label "GND"
-		(at 30.48 250.19 0)
-		(fields_autoplaced yes)
-		(effects
-			(font
-				(size 1.27 1.27)
-			)
-			(justify left bottom)
-		)
-	)
 	(label "3"
 		(at 208.28 34.29 180)
@@
 		)
 	)
-	(label "GND"
-		(at 59.69 252.73 0)
-		(fields_autoplaced yes)
-		(effects
-			(font
-				(size 1.27 1.27)
-			)
-			(justify left bottom)
-		)
-	)
 	(label "2"
 		(at 285.75 49.53 0)
@@
 		)
 	)
-	(label "GND"
-		(at 203.2 237.49 0)
-		(fields_autoplaced yes)
-		(effects
-			(font
-				(size 1.27 1.27)
-			)
-			(justify left bottom)
-		)
-	)
 	(label "6"
 		(at 358.14 35.56 270)
@@
 	)
 	(label "GND"
-		(at 304.8 101.6 0)
+		(at 302.26 101.6 0)
 		(fields_autoplaced yes)
 		(effects
@@
 		)
 	)
-	(label "GND"
-		(at 224.79 238.76 0)
-		(fields_autoplaced yes)
-		(effects
-			(font
-				(size 1.27 1.27)
-			)
-			(justify left bottom)
-		)
-	)
 	(label "SDA"
 		(at 227.33 139.7 0)
@@
 		)
 	)
-	(label "GND"
-		(at 330.2 232.41 0)
-		(fields_autoplaced yes)
-		(effects
-			(font
-				(size 1.27 1.27)
-			)
-			(justify left bottom)
-		)
-	)
 	(label "ADC4"
 		(at 247.65 177.8 0)
@@
 	(symbol
 		(lib_id "power:GND")
-		(at 30.48 251.46 0)
+		(at 30.48 247.65 0)
 		(unit 1)
 		(exclude_from_sim no)
@@
 		(fields_autoplaced yes)
 		(property "Reference" "#PWR01"
-			(at 30.48 257.81 0)
+			(at 30.48 254 0)
 			(effects
 				(font
@@
 		)
 		(property "Value" "GND"
-			(at 30.48 256.54 0)
+			(at 30.48 252.73 0)
 			(effects
 				(font
@@
 		)
 		(property "Footprint" ""
-			(at 30.48 251.46 0)
+			(at 30.48 247.65 0)
 			(effects
 				(font
@@
 		)
 		(property "Datasheet" ""
-			(at 30.48 251.46 0)
+			(at 30.48 247.65 0)
 			(effects
 				(font
@@
 		)
 		(property "Description" "Power symbol creates a global label with name \"GND\" , ground"
-			(at 30.48 251.46 0)
+			(at 30.48 247.65 0)
 			(effects
 				(font
@@
 	(symbol
 		(lib_id "power:GND")
-		(at 59.69 254 0)
+		(at 59.69 250.19 0)
 		(unit 1)
 		(exclude_from_sim no)
@@
 		(fields_autoplaced yes)
 		(property "Reference" "#PWR07"
-			(at 59.69 260.35 0)
+			(at 59.69 256.54 0)
 			(effects
 				(font
@@
 		)
 		(property "Value" "GND"
-			(at 59.69 259.08 0)
+			(at 59.69 255.27 0)
 			(effects
 				(font
@@
 		)
 		(property "Footprint" ""
-			(at 59.69 254 0)
+			(at 59.69 250.19 0)
 			(effects
 				(font
@@
 		)
 		(property "Datasheet" ""
-			(at 59.69 254 0)
+			(at 59.69 250.19 0)
 			(effects
 				(font
@@
 		)
 		(property "Description" "Power symbol creates a global label with name \"GND\" , ground"
-			(at 59.69 254 0)
+			(at 59.69 250.19 0)
 			(effects
 				(font
@@
 	(symbol
 		(lib_id "power:GND")
-		(at 203.2 240.03 0)
+		(at 203.2 234.95 0)
 		(unit 1)
 		(exclude_from_sim no)
@@
 		(fields_autoplaced yes)
 		(property "Reference" "#PWR019"
-			(at 203.2 246.38 0)
+			(at 203.2 241.3 0)
 			(effects
 				(font
@@
 		)
 		(property "Value" "GND"
-			(at 203.2 245.11 0)
+			(at 203.2 240.03 0)
 			(effects
 				(font
@@
 		)
 		(property "Footprint" ""
-			(at 203.2 240.03 0)
+			(at 203.2 234.95 0)
 			(effects
 				(font
@@
 		)
 		(property "Datasheet" ""
-			(at 203.2 240.03 0)
+			(at 203.2 234.95 0)
 			(effects
 				(font
@@
 		)
 		(property "Description" "Power symbol creates a global label with name \"GND\" , ground"
-			(at 203.2 240.03 0)
+			(at 203.2 234.95 0)
 			(effects
 				(font
