File: ATmega16U2.kicad_sch (KiCad schematic)
At the start: 28 parts, among them J1 Conn_02x02_Odd_Even, J11 Conn_02x03_Odd_Even, J12 USB_B, U3 ATmega16U2-A, Y3 ECS-160-20-4X-B-DN

Commit message: almost final
Parts:
- D7: footprint Diode_SMD:D_0402_1005Metric_Pad0.77x0.64mm_HandSolder -> Diode_SMD:D_0603_1608Metric
Changed lines of the file:
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@@
 			)
 		)
-		(property "Footprint" "Diode_SMD:D_0402_1005Metric_Pad0.77x0.64mm_HandSolder"
+		(property "Footprint" "Diode_SMD:D_0603_1608Metric"
 			(at 116.84 160.02 0)
 			(effects
