File: arduino-mega-2560.kicad_pcb (KiCad board)
At the start: 2 copper layers, 75 parts, among them J1 Conn_02x02_Odd_Even, J10 Conn_01x10, J11 Conn_02x03_Odd_Even, J12 USB_B, J15 Conn_02x03_Odd_Even, J2 PJ-031DH, J4 Conn_02x18_Odd_Even, J5 Conn_01x08, J6 Conn_01x08, J7 Conn_01x08, J8 Conn_01x08, J9 Conn_01x08, SW1 SW_MEC_5E, U1 LMV358, U2 LD1117S50CTR, U3 ATmega16U2-A, U4 MCU-ATMEGA2560-16AU_TQFP100_, U5 LP2985-3.3, U6 PMV48XP, Y1 CSTCE16M9V53-R0, Y2 Crystal

Commit message: last save attempt
Parts:
- J1: footprint Connector_Hirose:Hirose_DF11-4DP-2DSA_2x02_P2.00mm_Vertical -> Connector_PinHeader_1.00mm:PinHeader_2x02_P1.00mm_Vertical
- moved U1 114.3 mm to (192.5, 114.4)
- moved U6 94.1 mm to (192.6, 118.6)
- moved RV1 93.3 mm to (128.9, 97.3), turned to 90 degrees
- moved C10 93.0 mm to (160.0, 118.5)
- moved C1 92.4 mm to (193.4, 91.0)
- moved RV2 88.2 mm to (128.7, 108.7), turned to 90 degrees
- moved C18 82.8 mm to (150.2, 121.7)
- moved C11 79.3 mm to (201.4, 115.6)
- moved D7 77.1 mm to (149.0, 124.5)
- moved R21 67.9 mm to (139.8, 108.5)
- moved 1M1 66.0 mm to (145.0, 108.7)
- moved C13 66.0 mm to (139.8, 114.7)
- moved C14 66.0 mm to (139.8, 118.7)
- moved C17 66.0 mm to (139.8, 123.7)
- moved R14 66.0 mm to (145.0, 111.7)
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Routing:
- net +5V: track 0.00 -> 59.9 mm
- net /MCU-ATMEGA2560/ADC15: track 0.00 -> 35.4 mm
- net /MCU-ATMEGA2560/ADC14: track 0.00 -> 34.9 mm
- net /MCU-ATMEGA2560/ADC13: track 0.00 -> 34.4 mm
- net /MCU-ATMEGA2560/ADC12: track 0.00 -> 34.0 mm
- net /MCU-ATMEGA2560/ADC11: track 0.00 -> 33.8 mm
- net /MCU-ATMEGA2560/ADC10: track 0.00 -> 33.7 mm
- net /MCU-ATMEGA2560/ADC9: track 0.00 -> 33.4 mm
- net /MCU-ATMEGA2560/ADC8: track 0.00 -> 33.0 mm
- net /MCU-ATMEGA2560/ADC7: track 0.00 -> 30.7 mm
- net /MCU-ATMEGA2560/ADC6: track 0.00 -> 29.1 mm
- net /MCU-ATMEGA2560/ADC5: track 0.00 -> 28.8 mm
- net /MCU-ATMEGA2560/ADC4: track 0.00 -> 28.5 mm
- net /MCU-ATMEGA2560/ADC3: track 0.00 -> 28.4 mm
- net /MCU-ATMEGA2560/ADC2: track 0.00 -> 27.8 mm
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
Commit message: final top layer
Parts:
- moved C7 0.15 mm to (158.2, 96.4)
- moved R13 0.14 mm to (155.7, 100.5)
Routing:
- net +5V: track 59.9 -> 322.8 mm, vias 0 -> 1
- net /MCU-ATMEGA2560/3: track 0.00 -> 122.9 mm
- net /ATmega16U2/1: track 0.00 -> 100.4 mm
- net /MCU-ATMEGA2560/PC0: track 0.00 -> 88.6 mm
- net /MCU-ATMEGA2560/2: track 0.00 -> 73.6 mm
- net /ATmega16U2/USBVCC: track 0.00 -> 61.7 mm
- net /ATmega16U2/4: track 0.00 -> 55.2 mm
- net /ATmega16U2/USHIELD: track 0.00 -> 51.8 mm
- net Net-(D1-PadC): track 0.00 -> 40.7 mm
- net /MCU-ATMEGA2560/PA4: track 0.00 -> 40.6 mm
- net /ATmega16U2/RXL: track 0.00 -> 37.9 mm
- net /MCU-ATMEGA2560/PB7: track 0.00 -> 35.5 mm
- net /MCU-ATMEGA2560/PE5: track 0.00 -> 33.2 mm
- net Net-(U2-VIN): track 0.00 -> 31.3 mm
- net /MCU-ATMEGA2560/AREF: track 0.00 -> 29.5 mm
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Other:
- board outline added: 99.2 x 53.4 mm

Commit message: finished ratsnests connections
Parts:
- moved F1 1.23 mm to (118.9, 98.2)
Routing:
- net +5V: track 322.8 -> 490.0 mm, vias 1 -> 16
- net /MCU-ATMEGA2560/PB0: track 0.00 -> 106.6 mm, vias 0 -> 12
- net +3V3: track 0.00 -> 102.9 mm, vias 0 -> 2
- net /ATmega16U2/8: track 0.00 -> 83.3 mm, vias 0 -> 4
- net /MCU-ATMEGA2560/PB2: track 0.00 -> 81.9 mm, vias 0 -> 11
- net /MCU-ATMEGA2560/PC1: track 0.00 -> 81.3 mm, vias 0 -> 6
- net Net-(U4-VCC): track 6.47 -> 87.6 mm, vias 0 -> 8
- net /MCU-ATMEGA2560/PB1: track 0.00 -> 74.4 mm, vias 0 -> 13
- net /MCU-ATMEGA2560/PB3: track 0.00 -> 71.6 mm, vias 0 -> 10
- net /MCU-ATMEGA2560/PC3: track 0.00 -> 71.6 mm, vias 0 -> 4
- net /MCU-ATMEGA2560/PC5: track 0.00 -> 66.5 mm, vias 0 -> 2
- net /MCU-ATMEGA2560/PG1: track 0.00 -> 65.1 mm, vias 0 -> 4
- net /MCU-ATMEGA2560/PL6: track 0.00 -> 64.1 mm, vias 0 -> 9
- net /MCU-ATMEGA2560/PL5: track 0.00 -> 61.9 mm, vias 0 -> 6
- net /MCU-ATMEGA2560/PA6: track 0.00 -> 59.9 mm, vias 0 -> 2
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Other:
- board size 99.2 x 53.4 mm -> 109.3 x 53.4 mm

Commit message: instance before beginning to edit
Routing:
- net +5V: track 490.0 -> 490.6 mm
Other:
- board size 109.3 x 53.4 mm -> 104 x 53.4 mm
Changed lines of the file:
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@@
 	(gr_rect
 		(start 111.79 74.69)
-		(end 221.11 128.11)
+		(end 215.74 128.11)
 		(stroke
 			(width 0.05)
@@
 	)
 	(segment
+		(start 177 101.785686)
+		(end 178.044314 102.83)
+		(width 0.2)
+		(layer "F.Cu")
+		(net 2)
+	)
+	(segment
 		(start 161.37 86.23)
 		(end 161.38 86.24)
@@
 	)
 	(segment
-		(start 180.45 102.6)
-		(end 179.555687 102.6)
+		(start 177 98.91)
+		(end 177 101.785686)
 		(width 0.2)
 		(layer "F.Cu")
@@
 	)
 	(segment
-		(start 181.5 102.5)
-		(end 181.475 102.525)
-		(width 0.2)
-		(layer "F.Cu")
-		(net 2)
-	)
-	(segment
 		(start 161.4475 82.000424)
 		(end 161.4475 82.45)
@@
 	)
 	(segment
+		(start 179.555687 102.6)
+		(end 180.45 102.6)
+		(width 0.2)
+		(layer "F.Cu")
+		(net 2)
+	)
+	(segment
 		(start 140.45 125.24)
 		(end 144.955956 125.24)
@@
 	)
 	(segment
-		(start 179.325687 102.83)
-		(end 178.044314 102.83)
-		(width 0.2)
-		(layer "F.Cu")
-		(net 2)
-	)
-	(segment
 		(start 168 94)
 		(end 168 99.38)
@@
 		(start 158.0225 86.8575)
 		(end 156.88 88)
+		(width 0.2)
+		(layer "F.Cu")
+		(net 2)
+	)
+	(segment
+		(start 179.325687 102.83)
+		(end 179.555687 102.6)
 		(width 0.2)
 		(layer "F.Cu")
@@
 	)
 	(segment
+		(start 180.45 102.6)
+		(end 180.525 102.525)
+		(width 0.2)
+		(layer "F.Cu")
+		(net 2)
+	)
+	(segment
 		(start 177.43 98.48)
 		(end 177.43 97.230761)
@@
 	)
 	(segment
+		(start 178.044314 102.83)
+		(end 179.325687 102.83)
+		(width 0.2)
+		(layer "F.Cu")
+		(net 2)
+	)
+	(segment
 		(start 197.025785 102.64)
 		(end 197.106091 102.720305)
@@
 	)
 	(segment
-		(start 178.044314 102.83)
-		(end 177 101.785686)
-		(width 0.2)
-		(layer "F.Cu")
-		(net 2)
-	)
-	(segment
 		(start 207.98 114.849239)
 		(end 207.98 114.310761)
@@
 	)
 	(segment
-		(start 180.525 102.525)
-		(end 180.45 102.6)
+		(start 181.525 102.525)
+		(end 181.5 102.5)
 		(width 0.2)
 		(layer "F.Cu")
@@
 	)
 	(segment
-		(start 179.555687 102.6)
-		(end 179.325687 102.83)
-		(width 0.2)
-		(layer "F.Cu")
-		(net 2)
-	)
-	(segment
 		(start 168.15 122.639239)
 		(end 167.529239 123.26)
@@
 		(start 201.34 107.92)
 		(end 201.14 107.72)
-		(width 0.2)
-		(layer "F.Cu")
-		(net 2)
-	)
-	(segment
-		(start 177 101.785686)
-		(end 177 98.91)
 		(width 0.2)
 		(layer "F.Cu")
@@
 	)
 	(segment
+		(start 180.525 102.525)
+		(end 181.475 102.525)
+		(width 0.2)
+		(layer "F.Cu")
+		(net 2)
+	)
+	(segment
 		(start 115.26 122.33)
 		(end 128.75 122.33)
@@
 	)
 	(segment
+		(start 182.135 102.525)
+		(end 181.525 102.525)
+		(width 0.2)
+		(layer "F.Cu")
+		(net 2)
+	)
+	(segment
 		(start 168.784268 112.582795)
 		(end 168.874912 112.582795)
@@
 	)
 	(segment
+		(start 182.16 102.5)
+		(end 182.135 102.525)
+		(width 0.2)
+		(layer "F.Cu")
+		(net 2)
+	)
+	(segment
 		(start 139.46 105.51)
 		(end 140.275 105.51)
@@
 	)
 	(segment
-		(start 181.475 102.525)
-		(end 180.525 102.525)
-		(width 0.2)
-		(layer "F.Cu")
-		(net 2)
-	)
-	(segment
 		(start 139.275 123.74)
 		(end 139.14 123.605)
@@
 		(width 0.2)
 		(layer "F.Cu")
+		(net 2)
+	)
+	(segment
+		(start 181.475 102.525)
+		(end 181.5 102.5)
+		(width 0.2)
+		(layer "F.Cu")

Commit message: good progress
Parts:
- removed Y2: Crystal, Crystal:Crystal_SMD_HC49-SD_HandSoldering
- added RR1: 1M, Resistor_SMD:R_0201_0603Metric_Pad0.64x0.40mm_HandSolder, F.Cu at (125.1, 90.8)
- added Y3: ECS-160-20-4X-B-DN, ECS_160_20_4X_B_DN:XTAL_ECS-160-20-4X-B-DN, F.Cu at (131.7, 114.3)
- RV1, RV2: footprint Varistor:Varistor_Panasonic_VF -> Resistor_SMD:R_0201_0603Metric_Pad0.64x0.40mm_HandSolder
- SW1: footprint Button_Switch_SMD:SW_MEC_5GSH9 -> Button_Switch_SMD:SW_Push_1P1T_NO_CK_KSC6xxJ
- moved C1 59.3 mm to (138.7, 113.8), turned to -90 degrees
- moved C10 51.3 mm to (109.5, 109.2), turned to 90 degrees
- moved U6 51.0 mm to (142.2, 110.8), turned to 180 degrees
- moved J15 49.7 mm to (151.6, 98.9), turned to 180 degrees
- moved D1 46.6 mm to (111.6, 114.0), turned to 180 degrees
- moved U5 45.3 mm to (170.9, 119.7)
- moved C16 41.5 mm to (110.4, 94.8)
- moved R9 38.8 mm to (135.6, 123.8), turned to 90 degrees
- moved R11 38.7 mm to (156.0, 121.2)
- moved U2 38.6 mm to (115.0, 108.5)
- moved R1 34.8 mm to (152.8, 119.8), turned to 90 degrees
- moved C11 34.2 mm to (167.6, 120.5), turned to 180 degrees
- moved U1 33.9 mm to (158.7, 117.7), turned to -90 degrees
- moved D4 33.5 mm to (138.7, 109.5), turned to 90 degrees
- moved D7 32.7 mm to (137.2, 94.0), turned to 90 degrees
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Routing:
- net /MCU-ATMEGA2560/3: track 180.4 -> 76.1 mm, vias 5 -> 1
- net /MCU-ATMEGA2560/PC0: track 119.7 -> 26.2 mm
- net +3V3: track 102.9 -> 15.2 mm, vias 2 -> 0
- net /ATmega16U2/8: track 83.3 -> 1.99 mm, vias 4 -> 0
- net /ATmega16U2/4: track 89.1 -> 9.92 mm
- net /ATmega16U2/1: track 159.0 -> 81.0 mm, vias 8 -> 4
- net /ATmega16U2/USBVCC: track 100.1 -> 25.6 mm, vias 4 -> 0
- net /MCU-ATMEGA2560/PB0: track 106.6 -> 44.2 mm, vias 12 -> 1
- net /MCU-ATMEGA2560/PC1: track 81.3 -> 27.7 mm, vias 6 -> 0
- net /MCU-ATMEGA2560/PC3: track 71.6 -> 27.3 mm, vias 4 -> 1
- net /MCU-ATMEGA2560/PC5: track 66.5 -> 27.3 mm, vias 2 -> 1
- net +5V: track 490.6 -> 451.8 mm, vias 16 -> 8
- net /MCU-ATMEGA2560/PG1: track 65.1 -> 27.1 mm, vias 4 -> 0
- net /ATmega16U2/MISO2: track 59.2 -> 24.0 mm, vias 4 -> 2
- net Net-(U4-VCC): track 87.6 -> 53.3 mm, vias 8 -> 4
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- added copper zone on F.Cu, net +5V
Other:
- board size 104 x 53.4 mm -> 101.6 x 53.3 mm

Commit message: final edit
Parts:
- removed R19: 1K, Resistor_SMD:R_0201_0603Metric_Pad0.64x0.40mm_HandSolder
- moved C14 10.6 mm to (142.8, 113.9)
- moved R22 10.5 mm to (131.3, 87.2), turned to 180 degrees
- moved D5 9.52 mm to (143.6, 119.7)
- moved R14 5.08 mm to (132.2, 111.2)
- moved D4 4.74 mm to (142.3, 106.4)
- moved R21 3.46 mm to (131.3, 88.1), turned to 180 degrees
- moved R13 3.42 mm to (146.8, 117.4)
- moved U6 2.24 mm to (144.4, 110.8)
- moved D1 2.08 mm to (113.2, 115.3)
- moved C1 1.96 mm to (138.7, 115.7)
- moved C12 1.93 mm to (138.7, 118.0)
- moved R8 1.51 mm to (155.9, 116.2)
- moved RV1 1.46 mm to (130.1, 76.8)
- moved CR1 1.44 mm to (139.7, 123.1)
- moved R6 1.38 mm to (155.9, 117.2)
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Connections:
- C1 pad 2: +5V -> GND
- C10 pad 2: +5V -> GND
- C11 pad 2: +5V -> GND
- C12 pad 2: +5V -> GND
- C13 pad 1: /ATmega16U2/4 -> /ATmega16U2/DTR
- C14 pad 2: +5V -> GND
- C16 pad 2: +5V -> GND
- C17 pad 1: +5V -> GND
- C18 pad 1: +5V -> GND
- C2 pad 2: +5V -> GND
- C3 pad 2: +5V -> GND
- C4 pad 2: +5V -> GND
- C5 pad 2: +5V -> GND
- C6 pad 2: +5V -> GND
- C7 pad 2: +5V -> GND
- C8 pad 2: +5V -> GND
- C9 pad 2: +5V -> GND
- D4 pad 1: +5V -> GND
- D5 pad 1: +5V -> GND
- J10 pad 4: +5V -> GND
- J11 pad 6: +5V -> GND
- J15 pad 6: +5V -> GND
- J2 pad 1: +5V -> GND
- J2 pad 3: +5V -> GND
- J4 pad 35: +5V -> GND
- J4 pad 36: +5V -> GND
- J5 pad 6: +5V -> GND
- J5 pad 7: +5V -> GND
- JP1 pad 2: +5V -> GND
- R2 pad 2: +5V -> GND
- R8 pad 2: +5V -> GND
- SW1 pad 1: +5V -> GND
- SW1 pad 2: +5V -> GND
- U2 pad 1: +5V -> GND
- U3 pad 13: /ATmega16U2/4 -> /ATmega16U2/DTR
- U4 pad 11: +5V -> GND
- U4 pad 32: +5V -> GND
- U4 pad 62: +5V -> GND
- U4 pad 81: +5V -> GND
- U4 pad 99: +5V -> GND
- U5 pad 2: +5V -> GND
- Y1 pad 2: +5V -> GND
Routing:
- net +5V: track 451.8 -> 37.6 mm, vias 8 -> 10
- net GND: track 0.00 -> 71.7 mm, vias 0 -> 32
- net /ATmega16U2/D+: track 15.7 -> 41.9 mm, vias 0 -> 2
- net /ATmega16U2/DTR: track 0.00 -> 13.4 mm, vias 0 -> 2
- net /ATmega16U2/3: track 5.20 -> 18.2 mm
- net /MCU-ATMEGA2560/2: track 67.8 -> 57.6 mm
- net /ATmega16U2/RD-: track 19.9 -> 28.3 mm
- net /ATmega16U2/4: track 9.92 -> 1.80 mm, vias 2 -> 0
- net /MCU-ATMEGA2560/PB1: track 57.6 -> 62.1 mm, vias 1 -> 2
- net Net-(U4-VCC): track 53.3 -> 57.7 mm
- net /ATmega16U2/RD+: track 32.4 -> 28.3 mm
- net /MCU-ATMEGA2560/PB3: track 56.6 -> 59.5 mm
- net /MCU-ATMEGA2560/PC7: track 30.3 -> 27.6 mm
- net /ATmega16U2/USHIELD: track 32.5 -> 34.9 mm
- net /ATmega16U2/D-: track 21.3 -> 23.6 mm
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- added copper zone on B.Cu, net GND

Commit message: almost final
Parts:
- CR1: footprint CD1206_S01575:DIODE_CD1206-S01575_BRN -> Diode_SMD:D_0603_1608Metric
- D7: footprint Diode_SMD:D_0402_1005Metric_Pad0.77x0.64mm_HandSolder -> Diode_SMD:D_0603_1608Metric
- moved R1 1.83 mm to (151.3, 118.7)
- moved L2 1.15 mm to (158.1, 90.3)
- moved D7 0.38 mm to (137.3, 93.7)
Routing:
- net +5V: track 37.6 -> 20.8 mm, vias 10 -> 8
- net /ATmega16U2/D+: track 41.9 -> 31.1 mm, vias 2 -> 1
- net /ATmega16U2/D-: track 23.6 -> 31.0 mm, vias 2 -> 1
- net /ATmega16U2/RD+: track 28.3 -> 21.7 mm
- net /ATmega16U2/RD-: track 28.3 -> 21.8 mm
- net GND: track 71.7 -> 66.3 mm, vias 32 -> 31
- net /MCU-ATMEGA2560/ADC7: track 16.4 -> 18.9 mm
- net /ATmega16U2/1: track 80.2 -> 81.5 mm
- net /ATmega16U2/MISO2: track 23.5 -> 22.7 mm
- net /MCU-ATMEGA2560/AVCC: track 18.1 -> 18.8 mm
- net /MCU-ATMEGA2560/PB7: track 22.4 -> 21.8 mm
- net /MCU-ATMEGA2560/PB6: track 20.8 -> 21.4 mm
- net /MCU-ATMEGA2560/3: track 75.3 -> 74.7 mm
- net /MCU-ATMEGA2560/PG5: track 31.3 -> 30.8 mm
- net /MCU-ATMEGA2560/PH5: track 30.4 -> 29.9 mm
