File: arduino-mega-2560.kicad_pcb (KiCad board)
At the start: 2 copper layers, 101.6 x 53.3 mm, 80 parts, among them J1 Conn_02x02_Odd_Even, J10 Conn_01x10, J11 Conn_02x03_Odd_Even, J12 USB_B, J15 Conn_02x03_Odd_Even, J3 DCJ200-10-A-XX-K_REVA, J4 Conn_02x18_Odd_Even, J5 Conn_01x08, J6 Conn_01x08, J7 Conn_01x08, J8 Conn_01x08, J9 Conn_01x08, SW1 SW_MEC_5E, U1 LMV358, U2 LD1117S50CTR, U3 ATmega16U2-A, U4 MCU-ATMEGA2560-16AU_TQFP100_, U5 LP2985-3.3, U6 PMV48XP, Y1 CSTCE16M9V53-R0, Y3 ECS-160-20-4X-B-DN

Commit message: hardest trial
Parts:
- removed H1: MountingHole, MountingHole:MountingHole_3mm
- J4: footprint Connector_PinSocket_1.27mm:PinSocket_2x18_P1.27mm_Vertical -> Connector_PinSocket_2.00mm:PinSocket_2x18_P2.00mm_Vertical
- moved C12 29.6 mm to (166.4, 107.6), turned to -90 degrees
- moved C6 27.4 mm to (110.1, 99.1), turned to -90 degrees
- moved C5 26.9 mm to (177.2, 85.9), turned to 90 degrees
- moved C14 22.0 mm to (121.0, 111.1)
- moved C4 21.3 mm to (116.9, 106.6)
- moved C8 18.4 mm to (180.8, 98.3), turned to 0 degrees
- moved C7 17.9 mm to (166.7, 83.2)
- moved C2 15.0 mm to (165.6, 83.2), turned to 90 degrees
- moved C15 9.68 mm to (124.3, 103.8)
- moved R14 8.79 mm to (139.0, 105.6), turned to 0 degrees
- moved U2 7.24 mm to (116.3, 98.7), turned to 90 degrees
- moved J4 5.46 mm to (204.9, 82.7)
- moved L2 5.44 mm to (163.3, 88.8)
- moved C10 5.12 mm to (114.0, 104.2)
- moved C11 1.52 mm to (166.8, 119.3), turned to 90 degrees
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Connections:
- C8 pad 1: Net-(U4-VCC) -> +5V
- C9 pad 1: Net-(U4-VCC) -> +5V
- L2 pad 2: Net-(U4-VCC) -> +5V
- U4 pad 10: Net-(U4-VCC) -> +5V
- U4 pad 31: Net-(U4-VCC) -> +5V
- U4 pad 61: Net-(U4-VCC) -> +5V
Routing:
- net +5V: track 20.6 -> 328.2 mm, vias 8 -> 13
- net Net-(U4-VCC): track 57.3 -> 4.85 mm, vias 4 -> 0
- net Net-(U2-VIN): track 34.9 -> 17.2 mm
- net /ATmega16U2/3: track 18.2 -> 1.62 mm, vias 2 -> 0
- net /MCU-ATMEGA2560/AVCC: track 18.8 -> 7.18 mm, vias 2 -> 0
- net Net-(U3-UCAP): track 11.2 -> 1.65 mm
- net /MCU-ATMEGA2560/PL0: track 40.5 -> 47.0 mm, vias 2 -> 1
- net /ATmega16U2/1: track 86.1 -> 80.0 mm, vias 4 -> 2
- net /MCU-ATMEGA2560/PC7: track 27.6 -> 33.3 mm, vias 1 -> 0
- net /ATmega16U2/USBVCC: track 25.6 -> 31.1 mm
- net /MCU-ATMEGA2560/PL4: track 34.2 -> 39.7 mm, vias 3 -> 2
- net /MCU-ATMEGA2560/PB0: track 44.2 -> 49.4 mm, vias 1 -> 2
- net /MCU-ATMEGA2560/PH5: track 29.9 -> 35.0 mm
- net /MCU-ATMEGA2560/PB1: track 62.1 -> 67.1 mm, vias 2 -> 3
- net /MCU-ATMEGA2560/PB2: track 57.3 -> 61.9 mm, vias 1 -> 2
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- added copper zone on F.Cu, net +3V3
Other:
- board text added: "75"

Commit message: correction on pcb layout
Parts:
- added H1: MountingHole, MountingHole:MountingHole_3mm, F.Cu at (173.0, 136.4)
- J10: footprint Connector_PinSocket_1.00mm:PinSocket_1x10_P1.00mm_Vertical -> Connector_PinSocket_1.27mm:PinSocket_1x10_P1.27mm_Vertical
- J5, J6, J7, J8, J9: footprint Connector_PinSocket_1.00mm:PinSocket_1x08_P1.00mm_Vertical -> Connector_PinHeader_1.27mm:PinHeader_1x08_P1.27mm_Vertical
- U1: footprint Package_SO:MSOP-8-1EP_3x3mm_P0.65mm_EP2.5x3mm_Mask1.73x2.36mm_ThermalVias -> Package_SO:MSOP-8-1EP_3x3mm_P0.65mm_EP2.5x3mm_Mask1.73x2.36mm
- U4: footprint MCU-ATMEGA2560-16AU_TQFP100:TQFP100-0.5-14X14MM -> ATMEGA2560-16AU:QFP50P1600X1600X120-100N
- moved J6 5.15 mm to (189.6, 75.5)
- moved J7 3.79 mm to (180.2, 123.6)
- moved J10 1.95 mm to (153.7, 123.6)
- moved C12 1.95 mm to (166.1, 109.5), turned to 0 degrees
- moved L2 1.70 mm to (163.1, 87.1)
- moved C1 1.70 mm to (138.6, 114.0), turned to 90 degrees
- moved C11 1.40 mm to (166.8, 117.9)
- moved SW1 1.31 mm to (194.3, 117.4)
- moved J5 1.30 mm to (167.9, 123.6)
- moved C9 1.25 mm to (166.1, 108.5), turned to 0 degrees
- moved R3 0.89 mm to (168.4, 111.9)
- moved J9 0.52 mm to (168.3, 75.5)
Connections:
- C8 pad 1: +5V -> Net-(U4-VCC)
- C9 pad 1: +5V -> Net-(U4-VCC)
- L2 pad 2: +5V -> Net-(U4-VCC)
- U4 pad 10: +5V -> Net-(U4-VCC)
- U4 pad 31: +5V -> Net-(U4-VCC)
- U4 pad 61: +5V -> Net-(U4-VCC)
Routing:
- net Net-(U4-VCC): track 4.85 -> 63.1 mm, vias 0 -> 5
- net +5V: track 328.2 -> 300.1 mm, vias 13 -> 11
- net /MCU-ATMEGA2560/2: track 60.8 -> 76.1 mm, vias 0 -> 2
- net /MCU-ATMEGA2560/3: track 73.5 -> 81.6 mm
- net +3V3: track 17.7 -> 25.7 mm
- net /MCU-ATMEGA2560/ADC15: track 18.2 -> 26.0 mm
- net /MCU-ATMEGA2560/ADC14: track 18.0 -> 25.7 mm
- net /MCU-ATMEGA2560/ADC13: track 17.7 -> 24.2 mm
- net /MCU-ATMEGA2560/ADC12: track 17.5 -> 23.1 mm
- net /MCU-ATMEGA2560/ADC11: track 17.3 -> 22.7 mm
- net /MCU-ATMEGA2560/RXD1: track 19.4 -> 23.8 mm
- net /MCU-ATMEGA2560/TXD1: track 19.6 -> 24.0 mm
- net /MCU-ATMEGA2560/ADC10: track 17.1 -> 21.2 mm
- net /MCU-ATMEGA2560/ADC9: track 16.9 -> 20.9 mm
- net GND: track 68.7 -> 72.5 mm, vias 45 -> 32
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- added copper zone on F.Cu, net GND

Commit message: hopefully the final pcb layout
Parts:
- removed H1: MountingHole, MountingHole:MountingHole_3mm
Changed lines of the file:
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@@
 		(tags "resistor handsolder")
 		(property "Reference" "1M1"
-			(at 0 -1.05 90)
+			(at 0.0425 0.63 90)
 			(layer "F.SilkS")
 			(effects
@@
 			(at 0 -1.05 90)
 			(layer "F.SilkS")
+			(hide yes)
 			(effects
 				(font
@@
 			(at 0.225 1.09 90)
 			(layer "F.SilkS")
+			(hide yes)
 			(effects
 				(font
@@
 		(tags "resistor handsolder")
 		(property "Reference" "R14"
-			(at -0.3175 1.11 0)
+			(at -0.2325 -0.6 0)
 			(layer "F.SilkS")
 			(effects
@@
 			(at 6.76 -7.77 0)
 			(layer "F.SilkS")
+			(hide yes)
 			(effects
 				(font
@@
 		(tags "capacitor handsolder")
 		(property "Reference" "C12"
-			(at 0 -1.16 0)
+			(at -0.0325 1.3 0)
 			(layer "F.SilkS")
 			(effects
@@
 			(at 0.5625 0 0)
 			(layer "F.SilkS")
+			(hide yes)
 			(effects
 				(font
@@
 		(tags "resistor handsolder")
 		(property "Reference" "R5"
-			(at -3.8725 2.25 90)
+			(at -1.3725 0.85 90)
 			(layer "F.SilkS")
+			(hide yes)
 			(effects
 				(font
@@
 		)
 	)
-	(footprint "MountingHole:MountingHole_3mm"
-		(layer "F.Cu")
-		(at 173 136.4)
-		(descr "Mounting Hole 3mm, no annular")
-		(tags "mounting hole 3mm no annular")
-		(property "Reference" "H1"
-			(at 0 -4 0)
-			(layer "F.SilkS")
-			(effects
-				(font
-					(size 1 1)
-					(thickness 0.15)
-				)
-			)
-		)
-		(property "Value" "MountingHole"
-			(at 0 4 0)
-			(layer "F.Fab")
-			(effects
-				(font
-					(size 1 1)
-					(thickness 0.15)
-				)
-			)
-		)
-		(property "Footprint" "MountingHole:MountingHole_3mm"
-			(at 0 0 0)
-			(unlocked yes)
-			(layer "F.Fab")
-			(hide yes)
-			(effects
-				(font
-					(size 1.27 1.27)
-					(thickness 0.15)
-				)
-			)
-		)
-		(property "Datasheet" ""
-			(at 0 0 0)
-			(unlocked yes)
-			(layer "F.Fab")
-			(hide yes)
-			(effects
-				(font
-					(size 1.27 1.27)
-					(thickness 0.15)
-				)
-			)
-		)
-		(property "Description" "Mounting Hole without connection"
-			(at 0 0 0)
-			(unlocked yes)
-			(layer "F.Fab")
-			(hide yes)
-			(effects
-				(font
-					(size 1.27 1.27)
-					(thickness 0.15)
-				)
-			)
-		)
-		(property ki_fp_filters "MountingHole*")
-		(sheetname "Mounting Holes")
-		(sheetfile "mountingHoles.kicad_sch")
-		(attr exclude_from_pos_files exclude_from_bom)
-		(fp_circle
-			(center 0 0)
-			(end 3 0)
-			(stroke
-				(width 0.15)
-				(type solid)
-			)
-			(fill none)
-			(layer "Cmts.User")
-		)
-		(fp_circle
-			(center 0 0)
-			(end 3.25 0)
-			(stroke
-				(width 0.05)
-				(type solid)
-			)
-			(fill none)
-			(layer "F.CrtYd")
-		)
-		(fp_text user "${REFERENCE}"
-			(at 0 0 0)
-			(layer "F.Fab")
-			(effects
-				(font
-					(size 1 1)
-					(thickness 0.15)
-				)
-			)
-		)
-		(pad "" np_thru_hole circle
-			(at 0 0)
-			(size 3 3)
-			(drill 3)
-			(layers "*.Cu" "*.Mask")
-		)
-	)
 	(footprint "PMV48XP:SOT95P230X110-3N"
 		(layer "F.Cu")
 		(at 144.4478 110.7898 180)
 		(property "Reference" "U6"
-			(at 1.755395 -3.587085 0)
+			(at -3.1522 -0.4102 0)
 			(layer "F.SilkS")
+			(hide yes)
 			(effects
 				(font
@@
 			(at 3.9625 -0.31 0)
 			(layer "F.SilkS")
+			(hide yes)
 			(effects
 				(font
@@
 		(tags "capacitor handsolder")
 		(property "Reference" "C8"
-			(at 1.6325 -2 0)
+			(at -0.0325 -1 0)
 			(layer "F.SilkS")
 			(effects
@@
 		(tags "resistor handsolder")
 		(property "Reference" "R22"
-			(at 0 -1.05 0)
+			(at 0.1175 0.72 0)
 			(layer "F.SilkS")
 			(effects
@@
 		(tags "resistor handsolder")
 		(property "Reference" "R21"
-			(at 0 -1.05 0)
+			(at -1.7525 -0.86 0)
 			(layer "F.SilkS")
 			(effects
@@
 		(tags "capacitor handsolder")
 		(property "Reference" "C18"
-			(at 0 -1.16 0)
+			(at 2.8325 0 0)
 			(layer "F.SilkS")
 			(effects
@@
 		(tags "capacitor handsolder")
 		(property "Reference" "C16"
-			(at 0 -1.16 0)
+			(at 2.2875 0.65 0)
 			(layer "F.SilkS")
 			(effects
@@
 			(at 0 -1.05 90)
 			(layer "F.SilkS")
+			(hide yes)
 			(effects
 				(font
@@
 		(tags "capacitor handsolder")
 		(property "Reference" "C3"
-			(at 0 -1.16 0)
+			(at 1.7975 -0.03 0)
 			(layer "F.SilkS")
 			(effects
@@
 		(tags "resistor handsolder")
 		(property "Reference" "R6"
-			(at 0 -1.05 0)
+			(at -1.41 0.02 0)
 			(layer "F.SilkS")
+			(hide yes)
 			(effects
 				(font
@@
 		(tags "capacitor handsolder")
 		(property "Reference" "C7"
-			(at 0 -1.16 90)
+			(at -0.0325 1.3 90)
 			(layer "F.SilkS")
 			(effects
@@
 		(at 131.77 114.64)
 		(property "Reference" "Y3"
-			(at -2.597085 -3.637935 0)
+			(at 0 0 0)
 			(layer "F.SilkS")
+			(hide yes)
 			(effects
 				(font
@@
 		(at 113.16 112.67 180)
 		(property "Reference" "D1"
-			(at -0.127235 -2.671685 0)
+			(at 0 0 0)
 			(layer "F.SilkS")
 			(effects
@@
 		(tags "capacitor handsolder")
 		(property "Reference" "C2"
-			(at -0.0675 -1.1 90)
+			(at -0.0675 -1.4 90)
 			(layer "F.SilkS")
 			(effects
@@
 			(at 0 -1.43 90)
 			(layer "F.SilkS")
+			(hide yes)
 			(effects
 				(font
@@
 			(at 1.8925 1.9 0)
 			(layer "F.SilkS")
+			(hide yes)
 			(effects
 				(font
@@
 			(at 0 -1.16 90)
 			(layer "F.SilkS")
+			(hide yes)
 			(effects
 				(font
@@
 		(tags "LED handsolder")
 		(property "Reference" "D5"
-			(at 0 -1.05 90)
+			(at 0.02 -1.03 90)
 			(layer "F.SilkS")
 			(effects
@@
 			(at 0 -1.05 0)
 			(layer "F.SilkS")
+			(hide yes)
 			(effects
 				(font
@@
 		(tags "resistor handsolder")
 		(property "Reference" "R13"
-			(at 0.7325 -2.75 90)
+			(at 0.2075 -1 90)
 			(layer "F.SilkS")
 			(effects
@@
 		(tags "resistor handsolder")
 		(property "Reference" "R11"
-			(at 0 -1.05 0)
+			(at -5.16 -5.36 0)
 			(layer "F.SilkS")
+			(hide yes)
 			(effects
 				(font
@@
 		(tags "resistor handsolder")
 		(property "Reference" "R15"
-			(at 0 -1.05 90)
+			(at 0.4025 -1 90)
 			(layer "F.SilkS")
 			(effects
@@
 		(tags "capacitor handsolder")
 		(property "Reference" "C14"
-			(at 0 -1.16 0)
+			(at 0.2675 1 0)
 			(layer "F.SilkS")
 			(effects
@@
 		(tags "resistor handsolder")
 		(property "Reference" "RR1"
-			(at 0 -1.05 0)
+			(at 0.2225 -0.93 0)
 			(layer "F.SilkS")
 			(effects
@@
 		(layer "F.Cu")
 		(hatch edge 0.5)
+		(priority 12)
+		(connect_pads
+			(clearance 0.5)
+		)
+		(min_thickness 0.25)
+		(filled_areas_thickness no)
+		(fill yes
+			(thermal_gap 0.5)
+			(thermal_bridge_width 0.5)
+		)
+		(polygon
+			(pts
+				(xy 190.7 112.7) (xy 198.1 112.7) (xy 198.1 122.1) (xy 190.7 122.1)
+			)
+		)
+	)
+	(zone
+		(net 130)
+		(net_name "GND")
+		(layer "F.Cu")
+		(hatch edge 0.5)
 		(priority 2)
 		(connect_pads
@@
 			)
 		)
+	)
+	(zone
+		(net 2)
+		(net_name "+5V")
+		(layer "F.Cu")
+		(hatch edge 0.5)
+		(priority 11)
+		(connect_pads
+			(clearance 0.5)
+		)
+		(min_thickness 0.25)
+		(filled_areas_thickness no)
+		(fill yes
+			(thermal_gap 0.5)
+			(thermal_bridge_width 0.5)
+		)
+		(polygon
+			(pts
+				(xy 170.9 118) (xy 170.9 119.1) (xy 173.3 119.1) (xy 173.6 119.4) (xy 173.6 120) (xy 173.3 120.3)
+				(xy 171.1 120.3) (xy 171.1 121.1) (xy 170 122.2) (xy 170 122.9) (xy 178.7 122.9) (xy 178.7 121.3)
+				(xy 175.6 118.1)
+			)
+		)
