File: power-supply.kicad_sch (KiCad schematic)
At the start: 0 parts

Commit message: my potential final schematic
Parts:
- added C10: 100nF, symbol Device:C_Small
- added C4, C6: 47uF, symbol Device:C_Polarized
- added D1: M7, M7:DIOM505270X240, symbol M7:M7
- added J2: PJ-031DH, PJ-031DH:CUI_PJ-031DH, symbol PJ-031DH:PJ-031DH
- added U2: LD1117S50CTR, LD1117S50CTR:SOT230P700X180-4N, symbol LD1117S50CTR:LD1117S50CTR
Connections:
- new net: C10.1, C4.1, D1.C, U2.3 (VIN)
- new net: D1.A, J2.2
- new net +5V: C6.1, U2.2 (VOUT), U2.4 (VOUT__1)
- new net GND: C10.2, C4.2, C6.2, J2.1, J2.3, U2.1 (GND)
Other:
- company: (none) -> GEVITON ENTERPRISES LIMITED
- title: (none) -> POWER SUPPLY

Commit message: remaining with mh2029, the two connectors to finish footprint assignment
Parts:
- C10: footprint (none) -> Capacitor_SMD:C_0402_1005Metric_Pad0.74x0.62mm_HandSolder
- C4, C6: footprint (none) -> Capacitor_SMD:CP_Elec_4x3
- J2: footprint PJ-031DH:CUI_PJ-031DH -> PJ_031DH:CUI_PJ-031DH
Connections:
- net at C10.1, C4.1, U2.3 (VIN): now also D1.A; no longer D1.C
- net at J2.2: now also D1.C; no longer D1.A
Changed lines of the file:
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@@
-	)
-	(junction
-		(at 179.07 76.2)
-		(diameter 0)
-		(color 0 0 0 0)
 	)
 	(junction
@@
 	)
 	(junction
-		(at 179.07 78.74)
-		(diameter 0)
-		(color 0 0 0 0)
-	)
-	(junction
 		(at 114.3 76.2)
 		(diameter 0)
 		(color 0 0 0 0)
 	)
-	(wire
-		(pts
-			(xy 157.48 76.2) (xy 179.07 76.2)
+	(junction
+		(at 168.91 77.47)
+		(diameter 0)
+		(color 0 0 0 0)
+	)
+	(wire
+		(pts
+			(xy 168.91 68.58) (xy 168.91 77.47)
 		)
 		(stroke
@@
 	(wire
 		(pts
+			(xy 165.1 76.2) (xy 165.1 77.47)
+		)
+		(stroke
+			(width 0)
+			(type default)
+		)
+	)
+	(wire
+		(pts
 			(xy 64.77 76.2) (xy 71.12 76.2)
 		)
@@
 	(wire
 		(pts
-			(xy 157.48 78.74) (xy 179.07 78.74)
+			(xy 157.48 78.74) (xy 168.91 78.74)
 		)
 		(stroke
@@
 	(wire
 		(pts
-			(xy 179.07 78.74) (xy 179.07 76.2)
+			(xy 157.48 76.2) (xy 165.1 76.2)
 		)
 		(stroke
@@
 	(wire
 		(pts
+			(xy 165.1 77.47) (xy 168.91 77.47)
+		)
+		(stroke
+			(width 0)
+			(type default)
+		)
+	)
+	(wire
+		(pts
 			(xy 104.14 92.71) (xy 104.14 97.79)
 		)
@@
 	(wire
 		(pts
+			(xy 168.91 78.74) (xy 168.91 77.47)
+		)
+		(stroke
+			(width 0)
+			(type default)
+		)
+	)
+	(wire
+		(pts
 			(xy 86.36 81.28) (xy 86.36 76.2)
 		)
@@
 	(wire
 		(pts
+			(xy 179.07 77.47) (xy 168.91 77.47)
+		)
+		(stroke
+			(width 0)
+			(type default)
+		)
+	)
+	(wire
+		(pts
 			(xy 157.48 83.82) (xy 157.48 97.79)
 		)
@@
 	(wire
 		(pts
-			(xy 157.48 97.79) (xy 128.27 97.79)
-		)
-		(stroke
-			(width 0)
-			(type default)
-		)
-	)
-	(wire
-		(pts
-			(xy 179.07 76.2) (xy 179.07 73.66)
+			(xy 128.27 97.79) (xy 157.48 97.79)
+		)
+		(stroke
+			(width 0)
+			(type default)
+		)
+	)
+	(wire
+		(pts
+			(xy 179.07 78.74) (xy 179.07 77.47)
 		)
 		(stroke
@@
 			)
 		)
-		(property "Footprint" "PJ-031DH:CUI_PJ-031DH"
+		(property "Footprint" "PJ_031DH:CUI_PJ-031DH"
 			(at 52.07 76.2 0)
 			(effects
@@
 	(symbol
 		(lib_id "power:+5V")
-		(at 179.07 73.66 0)
+		(at 168.91 68.58 0)
 		(unit 1)
 		(exclude_from_sim no)
@@
 		(fields_autoplaced yes)
 		(property "Reference" "#PWR011"
-			(at 179.07 77.47 0)
+			(at 168.91 72.39 0)
 			(effects
 				(font
@@
 		)
 		(property "Value" "+5V"
-			(at 179.07 68.58 0)
+			(at 168.91 63.5 0)
 			(effects
 				(font
@@
 		)
 		(property "Footprint" ""
-			(at 179.07 73.66 0)
+			(at 168.91 68.58 0)
 			(effects
 				(font
@@
 		)
 		(property "Datasheet" ""
-			(at 179.07 73.66 0)
+			(at 168.91 68.58 0)
 			(effects
 				(font
@@
 		)
 		(property "Description" "Power symbol creates a global label with name \"+5V\""
-			(at 179.07 73.66 0)
+			(at 168.91 68.58 0)
 			(effects
 				(font
@@
 		(lib_id "M7:M7")
 		(at 91.44 76.2 0)
+		(mirror y)
 		(unit 1)
 		(exclude_from_sim no)
@@
 		(on_board yes)
 		(dnp no)
-		(fields_autoplaced yes)
 		(property "Reference" "D1"
 			(at 91.44 69.85 0)
@@
 			)
 		)
-		(property "Footprint" ""
+		(property "Footprint" "Capacitor_SMD:CP_Elec_4x3"
 			(at 180.0352 86.36 0)
 			(effects
@@
 			)
 		)
-		(property "Footprint" ""
+		(property "Footprint" "Capacitor_SMD:C_0402_1005Metric_Pad0.74x0.62mm_HandSolder"
 			(at 114.3 88.9 0)
 			(effects
@@
 			)
 		)
-		(property "Footprint" ""
+		(property "Footprint" "Capacitor_SMD:CP_Elec_4x3"
 			(at 103.1748 92.71 0)
 			(effects

Commit message: to edit in onshape
Parts:
- removed J2: PJ-031DH, PJ_031DH:CUI_PJ-031DH, symbol PJ-031DH:PJ-031DH
- added J3: DCJ200-10-A-XX-K_REVA, Connector_BarrelJack:BarrelJack_GCT_DCJ200-10-A_Horizontal, symbol DCJ200-10-A-XX-K_REVA:DCJ200-10-A-XX-K_REVA
Connections:
- net GND: now also J3.1, J3.3
- net at D1.C: now also J3.2
Changed lines of the file:
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@@
 	)
 	(symbol
-		(lib_id "PJ-031DH:PJ-031DH")
-		(at 52.07 76.2 0)
+		(lib_id "DCJ200-10-A-XX-K_REVA:DCJ200-10-A-XX-K_REVA")
+		(at 59.69 78.74 0)
 		(unit 1)
 		(exclude_from_sim no)
@@
 		(dnp no)
 		(fields_autoplaced yes)
-		(property "Reference" "J2"
-			(at 52.07 66.04 0)
-			(effects
-				(font
-					(size 1.27 1.27)
-				)
-			)
-		)
-		(property "Value" "PJ-031DH"
-			(at 52.07 68.58 0)
-			(effects
-				(font
-					(size 1.27 1.27)
-				)
-			)
-		)
-		(property "Footprint" "PJ_031DH:CUI_PJ-031DH"
-			(at 52.07 76.2 0)
+		(property "Reference" "J3"
+			(at 56.4543 69.85 0)
+			(effects
+				(font
+					(size 1.27 1.27)
+				)
+			)
+		)
+		(property "Value" "DCJ200-10-A-XX-K_REVA"
+			(at 56.4543 72.39 0)
+			(effects
+				(font
+					(size 1.27 1.27)
+				)
+			)
+		)
+		(property "Footprint" "Connector_BarrelJack:BarrelJack_GCT_DCJ200-10-A_Horizontal"
+			(at 59.69 78.74 0)
 			(effects
 				(font
@@
 		)
 		(property "Datasheet" ""
-			(at 52.07 76.2 0)
+			(at 59.69 78.74 0)
 			(effects
 				(font
@@
 		)
 		(property "Description" ""
-			(at 52.07 76.2 0)
-			(effects
-				(font
-					(size 1.27 1.27)
-				)
-				(hide yes)
-			)
-		)
-		(property "PARTREV" "1.05"
-			(at 52.07 76.2 0)
-			(effects
-				(font
-					(size 1.27 1.27)
-				)
-				(justify bottom)
-				(hide yes)
-			)
-		)
-		(property "MANUFACTURER" "CUI Devices"
-			(at 52.07 76.2 0)
-			(effects
-				(font
-					(size 1.27 1.27)
-				)
-				(justify bottom)
-				(hide yes)
-			)
-		)
-		(property "MAXIMUM_PACKAGE_HEIGHT" "7.5 mm"
-			(at 52.07 76.2 0)
+			(at 59.69 78.74 0)
+			(effects
+				(font
+					(size 1.27 1.27)
+				)
+				(hide yes)
+			)
+		)
+		(property "MF" "Global Connector Technology"
+			(at 59.69 78.74 0)
+			(effects
+				(font
+					(size 1.27 1.27)
+				)
+				(justify bottom)
+				(hide yes)
+			)
+		)
+		(property "MAXIMUM_PACKAGE_HEIGHT" "11 mm"
+			(at 59.69 78.74 0)
+			(effects
+				(font
+					(size 1.27 1.27)
+				)
+				(justify bottom)
+				(hide yes)
+			)
+		)
+		(property "Package" "None"
+			(at 59.69 78.74 0)
+			(effects
+				(font
+					(size 1.27 1.27)
+				)
+				(justify bottom)
+				(hide yes)
+			)
+		)
+		(property "Price" "None"
+			(at 59.69 78.74 0)
+			(effects
+				(font
+					(size 1.27 1.27)
+				)
+				(justify bottom)
+				(hide yes)
+			)
+		)
+		(property "Check_prices" "https://www.snapeda.com/parts/DCJ200-10-A-K1-K/Global+Connector+Technology/view-part/?ref=eda"
+			(at 59.69 78.74 0)
 			(effects
 				(font
@@
 		)
 		(property "STANDARD" "Manufacturer Recommendations"
-			(at 52.07 76.2 0)
+			(at 59.69 78.74 0)
+			(effects
+				(font
+					(size 1.27 1.27)
+				)
+				(justify bottom)
+				(hide yes)
+			)
+		)
+		(property "PARTREV" "A"
+			(at 59.69 78.74 0)
+			(effects
+				(font
+					(size 1.27 1.27)
+				)
+				(justify bottom)
+				(hide yes)
+			)
+		)
+		(property "SnapEDA_Link" "https://www.snapeda.com/parts/DCJ200-10-A-K1-K/Global+Connector+Technology/view-part/?ref=snap"
+			(at 59.69 78.74 0)
+			(effects
+				(font
+					(size 1.27 1.27)
+				)
+				(justify bottom)
+				(hide yes)
+			)
+		)
+		(property "MP" "DCJ200-10-A-K1-K"
+			(at 59.69 78.74 0)
+			(effects
+				(font
+					(size 1.27 1.27)
+				)
+				(justify bottom)
+				(hide yes)
+			)
+		)
+		(property "Purchase-URL" "https://www.snapeda.com/api/url_track_click_mouser/?unipart_id=641259&manufacturer=Global Connector Technology&part_name=DCJ200-10-A-K1-K&search_term=None"
+			(at 59.69 78.74 0)
+			(effects
+				(font
+					(size 1.27 1.27)
+				)
+				(justify bottom)
+				(hide yes)
+			)
+		)
+		(property "Description_1" "\nPower Barrel Connector Jack 2.05mm ID (0.081), 5.50mm OD (0.217) Through Hole, Right Angle\n"
+			(at 59.69 78.74 0)
+			(effects
+				(font
+					(size 1.27 1.27)
+				)
+				(justify bottom)
+				(hide yes)
+			)
+		)
+		(property "MANUFACTURER" "Global Connector Technology"
+			(at 59.69 78.74 0)
+			(effects
+				(font
+					(size 1.27 1.27)
+				)
+				(justify bottom)
+				(hide yes)
+			)
+		)
+		(property "Availability" "In Stock"
+			(at 59.69 78.74 0)
+			(effects
+				(font
+					(size 1.27 1.27)
+				)
+				(justify bottom)
+				(hide yes)
+			)
+		)
+		(property "SNAPEDA_PN" "DCJ200-10-A-K1-K"
+			(at 59.69 78.74 0)
 			(effects
 				(font
@@
 		(pin "1"
 		)
+		(pin "2"
+		)
 		(pin "3"
-		)
-		(pin "2"
 		)
 		(instances
 			(project ""
 				(path "/01593c05-32ee-43cc-9d3f-a6fed62a39f4/fa0a716f-64bc-4849-b74e-8fb50e8d1155"
-					(reference "J2")
+					(reference "J3")
 					(unit 1)
 				)
