File: mountingHoles.kicad_sch (KiCad schematic)
At the start: 5 parts

Commit message: correction on pcb layout
Parts:
- removed H1: MountingHole, MountingHole:MountingHole_3mm, symbol Mechanical:MountingHole
Changed lines of the file:
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@@
-		)
-	)
-	(symbol
-		(lib_id "Mechanical:MountingHole")
-		(at 87.63 50.8 0)
-		(unit 1)
-		(exclude_from_sim yes)
-		(in_bom no)
-		(on_board yes)
-		(dnp no)
-		(fields_autoplaced yes)
-		(property "Reference" "H1"
-			(at 90.17 49.5299 0)
-			(effects
-				(font
-					(size 1.27 1.27)
-				)
-				(justify left)
-			)
-		)
-		(property "Value" "MountingHole"
-			(at 90.17 52.0699 0)
-			(effects
-				(font
-					(size 1.27 1.27)
-				)
-				(justify left)
-			)
-		)
-		(property "Footprint" "MountingHole:MountingHole_3mm"
-			(at 87.63 50.8 0)
-			(effects
-				(font
-					(size 1.27 1.27)
-				)
-				(hide yes)
-			)
-		)
-		(property "Datasheet" "~"
-			(at 87.63 50.8 0)
-			(effects
-				(font
-					(size 1.27 1.27)
-				)
-				(hide yes)
-			)
-		)
-		(property "Description" "Mounting Hole without connection"
-			(at 87.63 50.8 0)
-			(effects
-				(font
-					(size 1.27 1.27)
-				)
-				(hide yes)
-			)
-		)
-		(instances
-			(project ""
-				(path "/01593c05-32ee-43cc-9d3f-a6fed62a39f4/0a7145a3-0ee0-45c1-ad79-b2107a4324b3"
-					(reference "H1")
-					(unit 1)
-				)
-			)
 		)
 	)
