File: components-demo/components-demo.kicad_sch (KiCad schematic)
At the start: 2 parts, among them U1 MCU-ATMEGA2560-16AU_TQFP100_

Commit message: updated schematic project
Parts:
- removed U1: MCU-ATMEGA2560-16AU_TQFP100_, MCU-ATMEGA2560-16AU_TQFP100_:TQFP100-0.5-14X14MM, symbol MCU-ATMEGA2560-16AU_SNAPMAGIC:MCU-ATMEGA2560-16AU_TQFP100_
- added U1: MCU-ATMEGA2560-16AU_TQFP100_, MCU-ATMEGA2560-16AU_TQFP100:TQFP100-0.5-14X14MM, symbol MCU-ATMEGA2560-16AU_TQFP100_:MCU-ATMEGA2560-16AU_TQFP100_

Commit message: done more work on schematic
Parts:
- removed U1: MCU-ATMEGA2560-16AU_TQFP100_, MCU-ATMEGA2560-16AU_TQFP100:TQFP100-0.5-14X14MM, symbol MCU-ATMEGA2560-16AU_TQFP100_:MCU-ATMEGA2560-16AU_TQFP100_
- added FB1: SMD-FERRITE-BEAD-30R-3A_0805_, SMD-FERRITE-BEAD-30R-3A_0805_:L0805, symbol SMD-FERRITE-BEAD-30R-3A_0805_:SMD-FERRITE-BEAD-30R-3A_0805_
- added J1: USB_B, symbol Connector:USB_B
- added U2: LD1117S50CTR, LD1117S50CTR:SOT230P700X180-4N, symbol LD1117S50CTR:LD1117S50CTR
- added U3: MCU-ATMEGA2560-16AU_TQFP100_, MCU-ATMEGA2560-16AU_TQFP100_:TQFP100-0.5-14X14MM, symbol MCU-ATMEGA2560-16AU_TQFP100_:MCU-ATMEGA2560-16AU_TQFP100_
- added U4: PMV48XP, PMV48XP:SOT95P230X110-3N, symbol PMV48XP:PMV48XP
- added Y1: CSTCE16M9V53-R0, CSTCE16M9V53-R0:OSC_CSTCE16M9V53-R0, symbol CSTCE16M9V53-R0:CSTCE16M9V53-R0
